Commit message: Pen training again w/Improved Model Geometry

File: PModel/PModel.urdf (robot description, URDF)
Before this commit: robot PModel, 9 links, 8 joints
Links:
- link Pen: geometry collision cylinder length=0.26218098 radius=0.005; visual mesh filename=meshes/Pen.stl scale=0.001 0.001 0.001
- link Ring: geometry collision box size=0.022 0.012 0.014; collision box size=0.022 0.012 0.014
Joints:
- joint Plate_Slider-7: limit lower=-0.055 upper=0.055 effort=1000000 velocity=1000000 -> lower=-0.015 upper=0.015 effort=1000000 velocity=1000000
- joint Slide_Slider-8: limit lower=-0.055 upper=0.055 effort=1000000 velocity=1000000 -> lower=-0.015 upper=0.015 effort=1000000 velocity=1000000

Commit message: A lot of carriage movement Still

File: PModel/PModel.urdf (robot description, URDF)
Before this commit: robot PModel, 9 links, 8 joints
Links:
- link Ring: geometry collision box size=0.026 0.018 0.065; collision box size=0.026 0.018 0.065
